Commit message: code update

File: agv_prbt/urdf/agv_prbt.xacro (robot description, xacro)
@@ -34,5 +34,5 @@
   <!-- connect the added tcp and the flange with a joint -->
   <joint name="prbt_fixed_joint_tcp" type="fixed">
-    <origin rpy="0 0 0" xyz="0 0 0.05"/>
+    <origin rpy="0 0 -0.785" xyz="0 0 0.05"/>
     <parent link="prbt_flange"/>
     <child link="prbt_tcp"/>
